Commit message: feat: hesai + utlidar 추가

File: go2_description/urdf/go2_description.urdf (robot description, URDF)
Before this commit: robot go2_description, 42 links, 41 joints
Links:
- added link hesai_lidar, mass 0.001; collision cylinder length=0.075 radius=0.05; visual cylinder length=0.075 radius=0.05
- added link utlidar_lidar, mass 0.001; collision cylinder length=0.04 radius=0.035; visual cylinder length=0.04 radius=0.035
Joints:
- added joint hesai_lidar_joint: type fixed, parent base, child hesai_lidar, origin xyz=0 0 0 rpy=0 0 0, axis 0 0 0
- added joint utlidar_lidar_joint: type fixed, parent base, child utlidar_lidar, origin xyz=0.28945 0 -0.046825 rpy=0 2.8782 0, axis 0 0 0

Commit message: feat: go2 sensor 데이터 받아오기 완료

File: go2_description/urdf/go2_description.urdf (robot description, URDF)
Before this commit: robot go2_description, 44 links, 43 joints
Links:
- added link Pandar64
- added link PandarXT-32
- added link base_link
- added link pandar
- added link rslidar
Joints:
- added joint base_link_to_base_joint: type fixed, parent base_link, child base, origin xyz=0 0 0 rpy=0 0 0, axis 0 0 0
- added joint hesai_pandar64_joint: type fixed, parent hesai_lidar, child Pandar64, origin xyz=0 0 0 rpy=0 0 0, axis 0 0 0
- added joint hesai_pandar_joint: type fixed, parent hesai_lidar, child pandar, origin xyz=0 0 0 rpy=0 0 0, axis 0 0 0
- added joint hesai_pandar_xt_joint: type fixed, parent hesai_lidar, child PandarXT-32, origin xyz=0 0 0 rpy=0 0 0, axis 0 0 0
- added joint hesai_rslidar_joint: type fixed, parent hesai_lidar, child rslidar, origin xyz=0 0 0 rpy=0 0 0, axis 0 0 0

Commit message: go2

File: go2_description/urdf/go2_description.urdf (robot description, URDF)
Before this commit: robot go2_description, 49 links, 48 joints
Joints:
- joint hesai_lidar_joint: origin xyz=0 0 0 rpy=0 0 0 -> xyz=0 0 0 rpy=0 0 1.5707963267948966

Commit message: go2 setup 완료

File: go2_description/urdf/go2_description.urdf (robot description, URDF)
Before this commit: robot go2_description, 49 links, 48 joints
Joints:
- joint hesai_lidar_joint: origin xyz=0 0 0 rpy=0 0 1.5707963267948966 -> xyz=0 0 0.15 rpy=0 0 1.5707963267948966

Commit message: base_link 및 state 소폭 수정

File: go2_description/urdf/go2_description.urdf (robot description, URDF)
Before this commit: robot go2_description, 49 links, 48 joints
Links:
- removed link base
- link base_link: mass None -> 6.921; geometry collision box size=0.3762 0.0935 0.114; visual mesh filename=package://go2_description/dae/base.dae
Joints:
- removed joint base_link_to_base_joint
- joint FL_hip_joint: parent base -> base_link
- joint FL_hip_rotor_joint: parent base -> base_link
- joint FR_hip_joint: parent base -> base_link
- joint FR_hip_rotor_joint: parent base -> base_link
- joint Head_upper_joint: parent base -> base_link
- joint RL_hip_joint: parent base -> base_link
- joint RL_hip_rotor_joint: parent base -> base_link
- joint RR_hip_joint: parent base -> base_link
- joint RR_hip_rotor_joint: parent base -> base_link
- joint front_camera_joint: parent base -> base_link
- joint hesai_lidar_joint: parent base -> base_link
- joint imu_joint: parent base -> base_link
- joint radar_joint: parent base -> base_link
- joint utlidar_lidar_joint: parent base -> base_link
